Commit message: Gazebo files only run in gazebo mode

File: robots/go2_description/xacro/robot.urdf.xacro (robot description, xacro)
@@ -1,135 +1,141 @@
 <?xml version="1.0"?>
 <robot name="go2" xmlns:xacro="http://www.ros.org/wiki/xacro">
-    <xacro:arg name="DEBUG" default="false"/>
-    <xacro:include filename="$(find go2_description)/xacro/const.xacro"/>
-    <xacro:include filename="$(find go2_description)/xacro/materials.xacro"/>
-    <xacro:include filename="$(find go2_description)/xacro/leg.xacro"/>
-    <!-- <xacro:include filename="$(find go2_description)/xacro/stairs.xacro"/> -->
-    <xacro:include filename="$(find go2_description)/xacro/gazebo.xacro"/>
-    <xacro:include filename="$(find go2_description)/xacro/ros2_control_macro.xacro"/>
-    <!-- <xacro:include filename="$(find go2_gazebo)/launch/stairs.urdf.xacro"/> -->
-    <!-- <xacro:stairs stairs="15" xpos="0" ypos="0" zpos="0" /> -->
-    <!-- Rotor related joint and link is only for demonstrate location. -->
-    <!-- Actually, the rotor will rotate and the joint is not fixed. Reduction ratio should be considered. -->
-    <!-- Debug mode will hung up the robot, use "true" or "false" to switch it. -->
-    <xacro:if value="$(arg DEBUG)">
-        <link name="world"/>
-        <joint name="base_static_joint" type="fixed">
+    <xacro:macro name="go2" params="mode">
+        <xacro:arg name="DEBUG" default="false"/>
+        <xacro:include filename="$(find go2_description)/xacro/const.xacro"/>
+        <xacro:include filename="$(find go2_description)/xacro/materials.xacro"/>
+        <xacro:include filename="$(find go2_description)/xacro/leg.xacro"/>
+        <!-- <xacro:include filename="$(find go2_description)/xacro/stairs.xacro"/> -->
+        <xacro:if value="${mode == 'gazebo'}">
+            <xacro:include filename="$(find go2_description)/xacro/gazebo.xacro"/>
+            <xacro:include filename="$(find go2_description)/xacro/ros2_control_macro.xacro"/>
+        </xacro:if>
+        <!-- <xacro:include filename="$(find go2_gazebo)/launch/stairs.urdf.xacro"/> -->
+        <!-- <xacro:stairs stairs="15" xpos="0" ypos="0" zpos="0" /> -->
+        <!-- Rotor related joint and link is only for demonstrate location. -->
+        <!-- Actually, the rotor will rotate and the joint is not fixed. Reduction ratio should be considered. -->
+        <!-- Debug mode will hung up the robot, use "true" or "false" to switch it. -->
+        <xacro:if value="$(arg DEBUG)">
+            <link name="world"/>
+            <joint name="base_static_joint" type="fixed">
+                <origin rpy="0 0 0" xyz="0 0 0"/>
+                <parent link="world"/>
+                <child link="base"/>
+            </joint>
+        </xacro:if>
+        <link name="base">
+            <visual>
+                <origin rpy="0 0 0" xyz="0 0 0"/>
+                <geometry>
+                    <box size="0.001 0.001 0.001"/>
+                </geometry>
+            </visual>
+        </link>
+        <joint name="floating_base" type="fixed">
             <origin rpy="0 0 0" xyz="0 0 0"/>
-            <parent link="world"/>
-            <child link="base"/>
+            <parent link="base"/>
+            <child link="trunk"/>
         </joint>
-    </xacro:if>
-    <link name="base">
-        <visual>
+        <link name="trunk">
+            <visual>
+                <origin rpy="0 0 0" xyz="0 0 0"/>
+                <geometry>
+                    <mesh filename="package://go2_description/meshes/trunk.dae" scale="1 1 1"/>
+                </geometry>
+                <!-- <material name="orange"/> -->
+            </visual>
+            <collision>
+                <origin rpy="0 0 0" xyz="0 0 0"/>
+                <geometry>
+                    <box size="${trunk_length} ${trunk_width} ${trunk_height}"/>
+                </geometry>
+            </collision>
+            <inertial>
+                <origin rpy="0 0 0" xyz="${trunk_com_x} ${trunk_com_y} ${trunk_com_z}"/>
+                <mass value="${trunk_mass}"/>
+                <inertia
+                    ixx="${trunk_ixx}" ixy="${trunk_ixy}" ixz="${trunk_ixz}"
+                    iyy="${trunk_iyy}" iyz="${trunk_iyz}"
+                    izz="${trunk_izz}"/>
+            </inertial>
+        </link>
+        <joint name="imu_joint" type="fixed">
+            <parent link="trunk"/>
+            <child link="imu_link"/>
             <origin rpy="0 0 0" xyz="0 0 0"/>
-            <geometry>
-                <box size="0.001 0.001 0.001"/>
-            </geometry>
-        </visual>
-    </link>
-    <joint name="floating_base" type="fixed">
-        <origin rpy="0 0 0" xyz="0 0 0"/>
-        <parent link="base"/>
-        <child link="trunk"/>
-    </joint>
-    <link name="trunk">
-        <visual>
+        </joint>
+        <link name="imu_link">
+            <inertial>
+                <mass value="0.001"/>
+                <origin rpy="0 0 0" xyz="0 0 0"/>
+                <inertia ixx="0.0001" ixy="0" ixz="0" iyy="0.0001" iyz="0" izz="0.0001"/>
+            </inertial>
+            <visual>
+                <origin rpy="0 0 0" xyz="0 0 0"/>
+                <geometry>
+                    <box size="0.001 0.001 0.001"/>
+                </geometry>
+                <!-- <material name="red"/> -->
+            </visual>
+            <collision>
+                <origin rpy="0 0 0" xyz="0 0 0"/>
+                <geometry>
+                    <box size=".001 .001 .001"/>
+                </geometry>
+            </collision>
+        </link>
+        <joint name="front_camera_joint" type="fixed">
+            <parent link="trunk"/>
+            <child link="front_camera"/>
+            <origin rpy="0 0 0" xyz="0.32715 -0.00003 0.04297"/>
+        </joint>
+        <link name="front_camera">
+        </link>
+        <!--
+        <joint name="load_joint" type="fixed">
+            <parent link="trunk"/>
+            <child link="load_link"/>
             <origin rpy="0 0 0" xyz="0 0 0"/>
-            <geometry>
-                <mesh filename="package://go2_description/meshes/trunk.dae" scale="1 1 1"/>
-            </geometry>
-            <!-- <material name="orange"/> -->
-        </visual>
-        <collision>
-            <origin rpy="0 0 0" xyz="0 0 0"/>
-            <geometry>
-                <box size="${trunk_length} ${trunk_width} ${trunk_height}"/>
-            </geometry>
-        </collision>
-        <inertial>
-            <origin rpy="0 0 0" xyz="${trunk_com_x} ${trunk_com_y} ${trunk_com_z}"/>
-            <mass value="${trunk_mass}"/>
-            <inertia
-                ixx="${trunk_ixx}" ixy="${trunk_ixy}" ixz="${trunk_ixz}"
-                iyy="${trunk_iyy}" iyz="${trunk_iyz}"
-                izz="${trunk_izz}"/>
-        </inertial>
-    </link>
-    <joint name="imu_joint" type="fixed">
-        <parent link="trunk"/>
-        <child link="imu_link"/>
-        <origin rpy="0 0 0" xyz="0 0 0"/>
-    </joint>
-    <link name="imu_link">
-        <inertial>
-            <mass value="0.001"/>
-            <origin rpy="0 0 0" xyz="0 0 0"/>
-            <inertia ixx="0.0001" ixy="0" ixz="0" iyy="0.0001" iyz="0" izz="0.0001"/>
-        </inertial>
-        <visual>
-            <origin rpy="0 0 0" xyz="0 0 0"/>
-            <geometry>
-                <box size="0.001 0.001 0.001"/>
-            </geometry>
-            <!-- <material name="red"/> -->
-        </visual>
-        <collision>
-            <origin rpy="0 0 0" xyz="0 0 0"/>
-            <geometry>
-                <box size=".001 .001 .001"/>
-            </geometry>
-        </collision>
-    </link>
-    <joint name="front_camera_joint" type="fixed">
-        <parent link="trunk"/>
-        <child link="front_camera"/>
-        <origin rpy="0 0 0" xyz="0.32715 -0.00003 0.04297"/>
-    </joint>
-    <link name="front_camera">
-    </link>
-    <!--
-    <joint name="load_joint" type="fixed">
-        <parent link="trunk"/>
-        <child link="load_link"/>
-        <origin rpy="0 0 0" xyz="0 0 0"/>
-    </joint>
-    <link name="load_link">
-        <inertial>
-            <mass value="5"/>
-            <origin rpy="0 0 0" xyz="0 0 0"/>
-            <inertia ixx="0.01" ixy="0" ixz="0" iyy="0.01" iyz="0" izz="0.01"/>
-        </inertial>
-        <visual>
-            <origin rpy="0 0 0" xyz="0 0 0.2"/>
-            <geometry>
-                <box size="0.5 0.3 0.2"/>
-            </geometry>
-        </visual>
-        <collision>
-            <origin rpy="0 0 0" xyz="0 0 0"/>
-            <geometry>
-                <box size=".001 .001 .001"/>
-            </geometry>
-        </collision>
-    </link>
--->
-    <xacro:leg name="FR" mirror="-1" mirror_dae= "False" front_hind="1"  front_hind_dae="True"  />
-    <xacro:leg name="FL" mirror="1"  mirror_dae="True"   front_hind="1"  front_hind_dae="True"  />
-    <xacro:leg name="RR" mirror="-1" mirror_dae="False"  front_hind="-1" front_hind_dae="False" />
-    <xacro:leg name="RL" mirror="1"  mirror_dae="True"   front_hind="-1" front_hind_dae="False" />
-    <xacro:go2_ros2_control interface_type="gazebo"/>
-        <!-- PosePublisher - P3D-equivalent -->
-    <xacro:macro name="go2_pose_publisher">
-      <gazebo>
-        <plugin filename="gz-sim-pose-publisher-system" name="gz::sim::systems::PosePublisher">
-          <publish_link_pose>false</publish_link_pose>
-          <publish_nested_model_pose>true</publish_nested_model_pose>
-          <publish_model_pose>true</publish_model_pose>
-          <update_frequency>30</update_frequency>
-          <use_pose_vector_msg>false</use_pose_vector_msg>
-        </plugin>
-      </gazebo>
+        </joint>
+        <link name="load_link">
+            <inertial>
+                <mass value="5"/>
+                <origin rpy="0 0 0" xyz="0 0 0"/>
+                <inertia ixx="0.01" ixy="0" ixz="0" iyy="0.01" iyz="0" izz="0.01"/>
+            </inertial>
+            <visual>
+                <origin rpy="0 0 0" xyz="0 0 0.2"/>
+                <geometry>
+                    <box size="0.5 0.3 0.2"/>
+                </geometry>
+            </visual>
+            <collision>
+                <origin rpy="0 0 0" xyz="0 0 0"/>
+                <geometry>
+                    <box size=".001 .001 .001"/>
+                </geometry>
+            </collision>
+        </link>
+    -->
+        <xacro:leg name="FR" mirror="-1" mirror_dae= "False" front_hind="1"  front_hind_dae="True"  />
+        <xacro:leg name="FL" mirror="1"  mirror_dae="True"   front_hind="1"  front_hind_dae="True"  />
+        <xacro:leg name="RR" mirror="-1" mirror_dae="False"  front_hind="-1" front_hind_dae="False" />
+        <xacro:leg name="RL" mirror="1"  mirror_dae="True"   front_hind="-1" front_hind_dae="False" />
+        <xacro:if value="${mode == 'gazebo'}">
+            <xacro:go2_ros2_control interface_type="gazebo"/>
+                <!-- PosePublisher - P3D-equivalent -->
+            <xacro:macro name="go2_pose_publisher">
+            <gazebo>
+                <plugin filename="gz-sim-pose-publisher-system" name="gz::sim::systems::PosePublisher">
+                <publish_link_pose>false</publish_link_pose>
+                <publish_nested_model_pose>true</publish_nested_model_pose>
+                <publish_model_pose>true</publish_model_pose>
+                <update_frequency>30</update_frequency>
+                <use_pose_vector_msg>false</use_pose_vector_msg>
+                </plugin>
+            </gazebo>
+            </xacro:macro>
+            <xacro:go2_pose_publisher />
+        </xacro:if>
     </xacro:macro>
-    <xacro:go2_pose_publisher />
 </robot>
